Commit message: first

File: common/engix_mod/urdf/engix_old.urdf (robot description, URDF)
Before this commit: robot engix, 24 links, 23 joints
Links:
- removed link base_footprint
- removed link camera_depth_frame
- removed link camera_depth_optical_frame
- removed link camera_link
- removed link camera_rgb_frame
- removed link camera_rgb_optical_frame
- removed link laser_tof
- added link lidar_tof_1; visual mesh filename=package://engix_description/meshes/lidar_tof_1.stl scale=0.001 0.001 0.001
Joints:
- removed joint base_footprint_joint
- removed joint camera_depth_joint
- removed joint camera_depth_optical_joint
- removed joint camera_joint
- removed joint camera_rgb_joint
- removed joint camera_rgb_optical_joint
- removed joint laser_tof_joint
- removed joint left_wheel_joint
- removed joint right_wheel_joint
- added joint left_wheel: type continuous, parent base_link, child lwheel, origin xyz=-0.133355 0.150817 0.079162 rpy=0 0 0, axis 0.0 1.0 -0.0
- added joint lidar_tof_joint: type fixed, parent base_link, child lidar_tof_1, origin xyz=0.157645 -0.04512 0.3677 rpy=0 0 0
- added joint right_wheel: type continuous, parent base_link, child rwheel, origin xyz=-0.133355 -0.146183 0.079162 rpy=0 0 0, axis 0.0 1.0 -0.0
