Commit message: camera frame fixed

File: common/engix_mod/urdf/engix.urdf (robot description, URDF)
Before this commit: robot engix, 18 links, 17 joints
Links:
- added link cameraLeft_depth_link
- added link cameraLeft_depth_link0
Joints:
- added joint cameraLeft_depth_joint: type fixed, parent ZED2_1, child cameraLeft_depth_link0, origin xyz=0 0 0 rpy=-1.57 0 0
- added joint cameraLeft_depth_joint1: type fixed, parent cameraLeft_depth_link0, child cameraLeft_depth_link, origin xyz=0 0 0 rpy=0 1.57 0

Commit message: ya

File: common/engix_mod/urdf/engix.urdf (robot description, URDF)
Before this commit: robot engix, 18 links, 17 joints
Links:
- added link camera_depth_frame
- added link camera_depth_optical_frame
- added link camera_link, mass 0.001
- added link camera_rgb_frame, mass 0.001
- added link camera_rgb_optical_frame
Joints:
- added joint camera_depth_joint: type fixed, parent camera_rgb_frame, child camera_depth_frame, origin xyz=0.176645 0.00992 0.4957 rpy=0 0 0
- added joint camera_depth_optical_joint: type fixed, parent camera_depth_frame, child camera_depth_optical_frame, origin xyz=0.176645 0.00992 0.4957 rpy=-1.5707 0 -1.5707
- added joint camera_joint: type fixed, parent camera_rgb_frame, child camera_link, origin xyz=0.176645 0.00992 0.4957 rpy=0 0 0
- added joint camera_rgb_joint: type fixed, parent base_link, child camera_rgb_frame, origin xyz=0.176645 0.00992 0.4957 rpy=0 0 0
- added joint camera_rgb_optical_joint: type fixed, parent camera_rgb_frame, child camera_rgb_optical_frame, origin xyz=0.176645 0.00992 0.4957 rpy=0 0 0
