Commit message: benewake tof initial

File: simulation/simulator_ws/src/tb_gazebo_description/robots/kobuki_hexagons_kinect.urdf.xacro (robot description, xacro)
@@ -17,8 +17,14 @@
   </xacro:hokuyo_utm30lx>
  -->
+<!--
   <xacro:include filename="$(find velodyne_description)/urdf/HDL-32E.urdf.xacro"/>
   <xacro:HDL-32E parent="base_link" name="velodyne" topic="/velodyne_points" hz="10" samples="440" gpu="${gpu}">
     <origin xyz="0 0 0.4" rpy="0 0 0" />
   </xacro:HDL-32E>
+ -->
+  <xacro:include filename="$(find ce30c_driver)/urdf/CE30C.urdf.xacro"/>
+  <xacro:CE30-C parent="base_link" name="velodyne" topic="/velodyne_points" hz="10" samples="440" gpu="${gpu}">
+    <origin xyz="0 0 0.4" rpy="0 0 0" />
+  </xacro:CE30-C>
   <xacro:kobuki/>
   <xacro:stack_hexagons parent="base_link"/>

Commit message: added gazebo gps plugin for turtlebot (default robot)

File: simulation/simulator_ws/src/tb_gazebo_description/robots/kobuki_hexagons_kinect.urdf.xacro (robot description, xacro)
@@ -3,36 +3,88 @@
     - Base      : kobuki
     - Stacks    : hexagons
-    - 3d Sensor : kinect
+    - 3d gps_sensor : kinect
 -->
-<robot name="turtlebot" xmlns:xacro="http://ros.org/wiki/xacro">
-  <gazebo>
-    <plugin name="p3d_base_controller" filename="libgazebo_ros_p3d.so">
-      <alwaysOn>true</alwaysOn>
-      <updateRate>50.0</updateRate>
-      <bodyName>base_link</bodyName>
-      <topicName>ground_truth/state</topicName>
-      <gaussianNoise>0.01</gaussianNoise>
-      <frameName>world</frameName>
-      <xyzOffsets>0 0 0</xyzOffsets>
-      <rpyOffsets>0 0 0</rpyOffsets>
-    </plugin>
-  </gazebo>
-  <xacro:arg name="gpu" default="false"/>
-  <xacro:property name="gpu" value="$(arg gpu)" />
-  <xacro:include filename="$(find tb_gazebo_description)/urdf/turtlebot_common_library.urdf.xacro" />
-  <xacro:include filename="$(find tb_gazebo_description)/urdf/kobuki.urdf.xacro" />
-  <xacro:include filename="$(find tb_gazebo_description)/urdf/stacks/hexagons.urdf.xacro"/>
-  <xacro:include filename="$(find tb_gazebo_description)/urdf/sensors/kinect.urdf.xacro"/>
-<!--   <xacro:include filename="$(find hector_sensors_description)/urdf/hokuyo_utm30lx.urdf.xacro" />
+<robot name="turtlebot"
+    xmlns:xacro="http://ros.org/wiki/xacro">
+    <gazebo>
+        <plugin name="p3d_base_controller" filename="libgazebo_ros_p3d.so">
+            <alwaysOn>true</alwaysOn>
+            <updateRate>50.0</updateRate>
+            <bodyName>base_link</bodyName>
+            <topicName>ground_truth/state</topicName>
+            <gaussianNoise>0.01</gaussianNoise>
+            <frameName>world</frameName>
+            <xyzOffsets>0 0 0</xyzOffsets>
+            <rpyOffsets>0 0 0</rpyOffsets>
+        </plugin>
+    </gazebo>
+    <xacro:arg name="gpu" default="false"/>
+    <xacro:property name="gpu" value="$(arg gpu)" />
+    <xacro:include filename="$(find tb_gazebo_description)/urdf/turtlebot_common_library.urdf.xacro" />
+    <xacro:include filename="$(find tb_gazebo_description)/urdf/kobuki.urdf.xacro" />
+    <xacro:include filename="$(find tb_gazebo_description)/urdf/stacks/hexagons.urdf.xacro"/>
+    <xacro:include filename="$(find tb_gazebo_description)/urdf/sensors/kinect.urdf.xacro"/>
+    <!--   <xacro:include filename="$(find hector_gps_sensors_description)/urdf/hokuyo_utm30lx.urdf.xacro" />
   <xacro:hokuyo_utm30lx name="laser" parent="base_link" ros_topic="scan" update_rate="40" ray_count="1040" min_angle="180" max_angle="-180">
     <origin xyz="0.00 0.00 0.20" rpy="0 0 0"/>
   </xacro:hokuyo_utm30lx>
  -->
-  <xacro:include filename="$(find velodyne_description)/urdf/HDL-32E.urdf.xacro"/>
-  <xacro:HDL-32E parent="base_link" name="velodyne" topic="/velodyne_points" hz="10" samples="440" gpu="${gpu}">
-    <origin xyz="0 0 0.4" rpy="0 0 0" />
-  </xacro:HDL-32E>
-  <xacro:kobuki/>
-  <xacro:stack_hexagons parent="base_link"/>
-  <xacro:sensor_kinect  parent="base_link"/>
+    <xacro:include filename="$(find velodyne_description)/urdf/HDL-32E.urdf.xacro"/>
+    <xacro:HDL-32E parent="base_link" name="velodyne" topic="/velodyne_points" hz="10" samples="440" gpu="${gpu}">
+        <origin xyz="0 0 0.4" rpy="0 0 0" />
+    </xacro:HDL-32E>
+    <!-- ================== GPS Sensor ================= -->
+    <xacro:property name="gps_height" value="0.2" />
+    <xacro:property name="gps_width" value="0.2" />
+    <joint name="fixed" type="fixed">
+        <parent link="base_link"/>
+        <child link="gps_sensor"/>
+    </joint>
+    <link name="gps_sensor">
+        <collision>
+            <origin xyz="0 0 ${gps_height/2}" rpy="0 0 0"/>
+            <geometry>
+                <box size="${gps_width} ${gps_width} ${gps_height}"/>
+            </geometry>
+        </collision>
+        <visual>
+            <origin xyz="0 0 ${gps_height/2}" rpy="0 0 0"/>
+            <geometry>
+                <box size="${gps_width} ${gps_width} ${gps_height}"/>
+            </geometry>
+            <material name="orange"/>
+        </visual>
+        <inertial>
+            <origin xyz="0 0 1" rpy="0 0 0"/>
+            <mass value="1"/>
+            <inertia ixx="1.0" ixy="0.0" ixz="0.0" iyy="1.0" iyz="0.0" izz="1.0"/>
+        </inertial>
+    </link>
+    <material name="orange">
+        <color rgba="${255/255} ${108/255} ${10/255} 1.0"/>
+    </material>
+    <gazebo reference="gps_sensor">
+        <material>Gazebo/Orange</material>
+    </gazebo>
+    <gazebo>
+        <plugin name="gazebo_ros_gps" filename="libhector_gazebo_ros_gps.so">
+            <updateRate>4.0</updateRate>
+            <bodyName>gps_sensor</bodyName>
+            <frameId>gps_sensor</frameId>
+            <topicName>/gps/fix</topicName>
+            <velocityTopicName>/gps/fix_velocity</velocityTopicName>
+            <referenceLatitude>55.16444</referenceLatitude>
+            <referenceLongitude>61.436844</referenceLongitude>
+            <referenceHeading>90</referenceHeading>
+            <referenceAltitude>10</referenceAltitude>
+            <offset>0 0 0</offset>
+            <drift>0.001 0.001 0.001</drift>
+            <gaussianNoise>0.05 0.05 0.05</gaussianNoise>
+            <velocityDrift>0.001 0.001 0.001</velocityDrift>
+            <velocityGaussianNoise>0.5 0.5 0.5</velocityGaussianNoise>
+        </plugin>
+    </gazebo>
+    <xacro:kobuki/>
+    <xacro:stack_hexagons parent="base_link"/>
+    <xacro:sensor_kinect parent="base_link"/>
 </robot>
